File: pcb/display.kicad_sch (KiCad schematic)
At the start: 3 parts, among them J1 Conn_01x40_MountingPin

Commit message: Placed components on PCB
Parts:
- removed C24: 10uF, Capacitor_THT:C_Disc_D5.0mm_W2.5mm_P2.50mm, symbol Device:C
- added C9: 10uF, Capacitor_SMD:C_0805_2012Metric_Pad1.18x1.45mm_HandSolder, symbol Device:C
- C23: footprint Capacitor_THT:C_Disc_D5.0mm_W2.5mm_P2.50mm -> Capacitor_SMD:C_0805_2012Metric_Pad1.18x1.45mm_HandSolder
- J1: footprint (none) -> Connector_FFC-FPC:Amphenol_F32R-1A7x1-11040_1x40-1MP_P0.5mm_Horizontal
Connections:
- net VCC is gone; now on net 3V3: C23.1, J1.12 (Pin_12), J1.38 (Pin_38), J1.39 (Pin_39), J1.6 (Pin_6), J1.7 (Pin_7)
- net GND: now also J1.34 (Pin_34), J1.35 (Pin_35), J1.36 (Pin_36), J1.MP (MountPin), C9.1
- net 3V3: now reaches J1.33 (Pin_33)
- net at C23.2: now also C9.2
- no-connect marks 0 -> 14
