File: pcb/inputs.kicad_sch (KiCad schematic)
At the start: 33 parts, among them J2 Conn_01x06_Pin, U11 74HC165, U12 74HC165

Commit message: Placed components on PCB
Parts:
- removed SWLB, SWRB: SW_DPST, ray:SW_PUSH_6mm, symbol Switch:SW_DPST
- added R21: 10k, Resistor_SMD:R_0805_2012Metric_Pad1.20x1.40mm_HandSolder, symbol Device:R
- added SWLB1, SWRB1: ESPRST, ray:SW_SIDE_PUSH_3x6mm, symbol Switch:SW_DPST_x2
- added SWRST1: SW_DPST, ray:SW_PUSH_6mm, symbol Switch:SW_DPST
- C25, C26: footprint Capacitor_THT:C_Disc_D5.0mm_W2.5mm_P2.50mm -> Capacitor_SMD:C_0805_2012Metric_Pad1.18x1.45mm_HandSolder
- R1, R10, R11, R12, R13, R14, R15, R16, R2, R3, R4, R5, R6, R7, R8, R9: footprint Resistor_THT:R_Axial_DIN0204_L3.6mm_D1.6mm_P5.08mm_Horizontal -> Resistor_SMD:R_0805_2012Metric_Pad1.20x1.40mm_HandSolder
- renumbered SWA to SWA1, SWB to SWB1, SWD to SWD1, SWL to SWL1, SWMENU to SWMENU1, SWR to SWR1, SWSTART to SWSTART1, SWU to SWU1, SWX to SWX1, SWY to SWY1
Connections:
- net BTNLB: now also SWLB1.2 (B)
- net BTNRB: now also SWRB1.2 (B)
- net GND: now also SWLB1.1 (A), SWRB1.1 (A), SWRST1.1
- new net 5V: R21.1
- new net BTNRST: R21.2, SWRST1.4
- no-connect marks 0 -> 25
