File: pcb/mud-16.kicad_sch (KiCad schematic)
At the start: 15 parts, among them U1 74LVC1G04, U10 74HC595, U3 Tang_Nano_9K, U6 AS7C3513B, U9 74HC595

Commit message: Placed components on PCB
Parts:
- removed C37: 10uF, Capacitor_THT:C_Disc_D5.0mm_W2.5mm_P2.50mm, symbol Device:C
- added C24: 10uF, Capacitor_SMD:C_0805_2012Metric_Pad1.18x1.45mm_HandSolder, symbol Device:C
- added R22, R23: 10k, Resistor_SMD:R_0805_2012Metric_Pad1.20x1.40mm_HandSolder, symbol Device:R
- C19, C20, C21, C22, C33, C34, C35, C36: footprint Capacitor_THT:C_Disc_D5.0mm_W2.5mm_P2.50mm -> Capacitor_SMD:C_0805_2012Metric_Pad1.18x1.45mm_HandSolder
- U10, U9: footprint Package_DIP:DIP-16_W7.62mm -> Package_SO:SOIC-16_3.9x9.9mm_P1.27mm
Connections:
- net 5V: now also C36.1, CPU1.17 (~{HALT}), CPU1.21 (~{VPA}), CPU1.22 (~{BERR}), CPU1.23 (~{IPL2}), CPU1.24 (~{IPL1}), CPU1.25 (~{IPL0}), U3.31 (5V)
- net GND: now also C24.1, R22.2, R23.2
- net LDS: now also R23.1
- net R/W: now also U3.48 (63_IOR5A)
- net UDS: now also R22.1
- net 1V8_CPU_OE: now reaches U3.45 (84_IOT10A_1V8)
- net 1V8_CLK: now reaches U3.46 (85_IOT8B_1V8)
- net 1V8_LED: now reaches U3.47 (86_IOT8A_1V8)
- net at C33.2: now also C24.2; no longer C34.1
- net at C36.2: now also C34.1
- net CLK: now reaches CPU1.15 (CLK)
- net BTNRST: now reaches CPU1.18 (~{RESET})
- net CPU A1 renamed CPU_A1
- net CPU A10 renamed CPU_A10
- net CPU A11 renamed CPU_A11
- net CPU A12 renamed CPU_A12
- net CPU A13 renamed CPU_A13
- net CPU A14 renamed CPU_A14
- net CPU A15 renamed CPU_A15
- net CPU A16 renamed CPU_A16
- net CPU A2 renamed CPU_A2
- net CPU A3 renamed CPU_A3
- net CPU A4 renamed CPU_A4
- net CPU A5 renamed CPU_A5
- net CPU A6 renamed CPU_A6
- net CPU A7 renamed CPU_A7
- net CPU A8 renamed CPU_A8
- net CPU A9 renamed CPU_A9
- net CPU AS renamed CPU_AS
- net CPU BG renamed CPU_BG
- net CPU BGACK renamed CPU_BGACK
- net CPU BR renamed CPU_BR
- net CPU D0 renamed CPU_D0
- net CPU D1 renamed CPU_D1
- net CPU D10 renamed CPU_D10
- net CPU D11 renamed CPU_D11
- net CPU D12 renamed CPU_D12
- net CPU D13 renamed CPU_D13
- net CPU D14 renamed CPU_D14
- net CPU D15 renamed CPU_D15
- net CPU D2 renamed CPU_D2
- net CPU D3 renamed CPU_D3
- net CPU D4 renamed CPU_D4
- net CPU D5 renamed CPU_D5
- net CPU D6 renamed CPU_D6
- net CPU D7 renamed CPU_D7
- net CPU D8 renamed CPU_D8
- net CPU D9 renamed CPU_D9
- net CPU DTACK renamed CPU_DTACK
- net CPU LDS renamed CPU_LDS
- net CPU R/W renamed CPU_R/W
- net CPU UDS renamed CPU_UDS
- no-connect marks 7 -> 14
Other:
- added sheet Power Sheet (power.kicad_sch)
- note removed: "FIGURE OUT MEMORY IN FPGA LATER!!!"
- note removed: "FIGURE OUT POWER"
- note removed: "Logic Shifters"
- note removed: "a ton of stuff needs caps and resistors and stuff including logic shifters and cpu and ram and fpga and everything"
- moved on the sheet: C36

Commit message: routing pcb
Connections:
- net A12: now also U10.6 (QG); no longer U10.3 (QD)
- net A13: now also U10.5 (QF); no longer U10.4 (QE)
- net A14: now also U10.4 (QE); no longer U10.5 (QF)
- net A15: now also U10.3 (QD); no longer U10.6 (QG)
- net D0: now also U3.8 (28_IOB11B); no longer U3.1 (38_IOB31B)
- net D1: now also U3.7 (27_IOB11A); no longer U3.2 (37_IOB31A)
- net D2: now also U3.6 (26_IOB8B); no longer U3.3 (36_IOB29B)
- net D3: now also U3.5 (25_IOB8A); no longer U3.4 (39_IOB33A)
- net D4: now also U3.4 (39_IOB33A); no longer U3.5 (25_IOB8A)
- net D5: now also U3.3 (36_IOB29B); no longer U3.6 (26_IOB8B)
- net D6: now also U3.2 (37_IOB31A); no longer U3.7 (27_IOB11A)
- net D7: now also U3.1 (38_IOB31B); no longer U3.8 (28_IOB11B)
- net A16: no longer names the net of U10.7 (QH)
- net CPU_A16: no longer names the net of CPU1.44 (A16)
- no-connect marks 14 -> 16
Changed lines of the file:
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@@
 	)
 	(no_connect
+		(at 265.43 116.84)
+	)
+	(no_connect
 		(at 85.09 74.93)
 	)
@@
 	)
 	(no_connect
+		(at 85.09 67.31)
+	)
+	(no_connect
 		(at 54.61 67.31)
 	)
@@
 	(wire
 		(pts
-			(xy 86.36 67.31) (xy 85.09 67.31)
-		)
-		(stroke
-			(width 0)
-			(type default)
-		)
-	)
-	(wire
-		(pts
 			(xy 107.95 158.75) (xy 109.22 158.75)
 		)
@@
 		)
 	)
-	(global_label "D6"
+	(global_label "D1"
 		(shape input)
 		(at 162.56 71.12 180)
@@
 		)
 	)
-	(global_label "D0"
+	(global_label "D7"
 		(shape input)
 		(at 162.56 55.88 180)
@@
 		)
 	)
-	(global_label "D5"
+	(global_label "D2"
 		(shape input)
 		(at 162.56 68.58 180)
@@
 		)
 	)
-	(global_label "CPU_A16"
-		(shape input)
-		(at 86.36 67.31 0)
-		(fields_autoplaced yes)
-		(effects
-			(font
-				(size 1.27 1.27)
-			)
-			(justify left)
-		)
-		(property "Intersheetrefs" "${INTERSHEET_REFS}"
-			(at 97.6909 67.31 0)
-			(effects
-				(font
-					(size 1.27 1.27)
-				)
-				(justify left)
-				(hide yes)
-			)
-		)
-	)
 	(global_label "D11"
 		(shape input)
@@
 		)
 	)
-	(global_label "A14"
+	(global_label "A13"
 		(shape input)
 		(at 265.43 111.76 0)
@@
 		)
 	)
-	(global_label "D2"
+	(global_label "D5"
 		(shape input)
 		(at 162.56 60.96 180)
@@
 		)
 	)
-	(global_label "A12"
+	(global_label "A15"
 		(shape input)
 		(at 265.43 106.68 0)
@@
 		)
 	)
-	(global_label "A16"
-		(shape input)
-		(at 265.43 116.84 0)
-		(fields_autoplaced yes)
-		(effects
-			(font
-				(size 1.27 1.27)
-			)
-			(justify left)
-		)
-		(property "Intersheetrefs" "${INTERSHEET_REFS}"
-			(at 271.9228 116.84 0)
-			(effects
-				(font
-					(size 1.27 1.27)
-				)
-				(justify left)
-				(hide yes)
-			)
-		)
-	)
 	(global_label "CPU_BG"
 		(shape input)
@@
 		)
 	)
-	(global_label "D7"
+	(global_label "D0"
 		(shape input)
 		(at 162.56 73.66 180)
@@
 		)
 	)
-	(global_label "D3"
+	(global_label "D4"
 		(shape input)
 		(at 162.56 63.5 180)
@@
 		)
 	)
-	(global_label "D1"
+	(global_label "D6"
 		(shape input)
 		(at 162.56 58.42 180)
@@
 		)
 	)
-	(global_label "D4"
+	(global_label "D3"
 		(shape input)
 		(at 162.56 66.04 180)
@@
 		)
 	)
-	(global_label "A13"
+	(global_label "A14"
 		(shape input)
 		(at 265.43 109.22 0)
@@
 		)
 	)
-	(global_label "A15"
+	(global_label "A12"
 		(shape input)
 		(at 265.43 114.3 0)
