File: pcb/logicshifters.kicad_sch (KiCad schematic)
At the start: 37 parts, among them U13 SN74LVC8T245, U14 SN74LVC8T245, U15 74LVC1G04, U16 SN74LVC8T245, U2 SN74LVC8T245, U4 SN74LVC8T245, U5 SN74LVC8T245, U7 SN74LVC8T245, U8 SN74LVC8T245

Commit message: Placed components on PCB
Parts:
- removed C7, C8: 0.1uF, Capacitor_THT:C_Disc_D5.0mm_W2.5mm_P2.50mm, symbol Device:C
- removed C9: 1uF, Capacitor_THT:C_Disc_D5.0mm_W2.5mm_P2.50mm, symbol Device:C
- removed U16: SN74LVC8T245, Package_SO:TSSOP-24_4.4x7.8mm_P0.65mm, symbol Logic_LevelTranslator:SN74LVC8T245
- added C39: 0.1uF, Capacitor_SMD:C_0805_2012Metric_Pad1.18x1.45mm_HandSolder, symbol Device:C
- added C40: 10uF, Capacitor_SMD:C_0805_2012Metric_Pad1.18x1.45mm_HandSolder, symbol Device:C
- added D1: WS2812B, LED_SMD:LED_WS2812B_PLCC4_5.0x5.0mm_P3.2mm, symbol LED:WS2812B
- added R24: 330, Resistor_SMD:R_0805_2012Metric_Pad1.20x1.40mm_HandSolder, symbol Device:R
- C1, C10, C11, C12, C13, C14, C15, C16, C17, C18, C2, C27, C28, C29, C3, C30, C31, C32, C4, C5, C6: footprint Capacitor_THT:C_Disc_D5.0mm_W2.5mm_P2.50mm -> Capacitor_SMD:C_0805_2012Metric_Pad1.18x1.45mm_HandSolder
- R17, R18, R19, R20: footprint Resistor_THT:R_Axial_DIN0204_L3.6mm_D1.6mm_P5.08mm_Horizontal -> Resistor_SMD:R_0805_2012Metric_Pad1.20x1.40mm_HandSolder
Connections:
- net 1V8: now also U14.2 (DIR)
- net 3V3: no longer C29.1, U14.2 (DIR), U14.23 (V_{CCB}), U14.24 (V_{CCB}), U5.2 (DIR), U7.2 (DIR), U8.2 (DIR)
- net 5V: now also C29.1, U14.23 (V_{CCB}), U14.24 (V_{CCB}), U5.2 (DIR), U7.2 (DIR), U8.2 (DIR), C40.2
- net GND: now also D1.3 (VSS); no longer U14.16 (B6), U14.17 (B5), U14.18 (B4), U14.6 (A4), U14.7 (A5), U14.8 (A6), U8.16 (B6), U8.8 (A6)
- net BGACK renamed CPU_BGACK
- net BR renamed CPU_BR
- net CPU A1 renamed CPU_A1
- net CPU A10 renamed CPU_A10
- net CPU A11 renamed CPU_A11
- net CPU A12 renamed CPU_A12
- net CPU A13 renamed CPU_A13
- net CPU A14 renamed CPU_A14
- net CPU A15 renamed CPU_A15
- net CPU A16 renamed CPU_A16
- net CPU A2 renamed CPU_A2
- net CPU A3 renamed CPU_A3
- net CPU A4 renamed CPU_A4
- net CPU A5 renamed CPU_A5
- net CPU A6 renamed CPU_A6
- net CPU A7 renamed CPU_A7
- net CPU A8 renamed CPU_A8
- net CPU A9 renamed CPU_A9
- net CPU AS renamed CPU_AS
- net CPU BG renamed CPU_BG
- net CPU D0 renamed CPU_D0
- net CPU D1 renamed CPU_D1
- net CPU D10 renamed CPU_D10
- net CPU D11 renamed CPU_D11
- net CPU D12 renamed CPU_D12
- net CPU D13 renamed CPU_D13
- net CPU D14 renamed CPU_D14
- net CPU D15 renamed CPU_D15
- net CPU D2 renamed CPU_D2
- net CPU D3 renamed CPU_D3
- net CPU D4 renamed CPU_D4
- net CPU D5 renamed CPU_D5
- net CPU D6 renamed CPU_D6
- net CPU D7 renamed CPU_D7
- net CPU D8 renamed CPU_D8
- net CPU D9 renamed CPU_D9
- net CPU LDS renamed CPU_LDS
- net CPU OE renamed CPU_OE
- net CPU_OE: now also U14.18 (B4), U8.8 (A6)
- net CPU R/W renamed CPU_R/W
- net CPU UDS renamed CPU_UDS
- net DTACK renamed CPU_DTACK
- new net: C39.1, D1.1 (VDD)
- new net: C39.2, C40.1
- new net: R24.2, U14.16 (B6)
- new net: D1.4 (DIN), R24.1
- new net 1V8_CLK: U14.7 (A5)
- new net 1V8_CPU_OE: U14.6 (A4)
- new net 1V8_LED: U14.8 (A6)
- new net CLK: U14.17 (B5)
- no-connect marks 0 -> 1
Other:
- moved on the sheet: C28, C29, C30, U14

Commit message: routing pcb
Connections:
- net A16 is gone; now on net GND: U5.14 (B8)
- net CPU_A16 is gone; now on net GND: U5.10 (A8)
Changed lines of the file:
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@@
 		)
 	)
-	(global_label "CPU_A16"
-		(shape input)
-		(at 179.07 85.09 180)
-		(fields_autoplaced yes)
-		(effects
-			(font
-				(size 1.27 1.27)
-			)
-			(justify right)
-		)
-		(property "Intersheetrefs" "${INTERSHEET_REFS}"
-			(at 167.7391 85.09 0)
-			(effects
-				(font
-					(size 1.27 1.27)
-				)
-				(justify right)
-				(hide yes)
-			)
-		)
-	)
 	(global_label "A13"
 		(shape output)
@@
 		)
 	)
-	(global_label "A16"
-		(shape output)
-		(at 201.93 85.09 0)
-		(fields_autoplaced yes)
-		(effects
-			(font
-				(size 1.27 1.27)
-			)
-			(justify left)
-		)
-		(property "Intersheetrefs" "${INTERSHEET_REFS}"
-			(at 208.4228 85.09 0)
-			(effects
-				(font
-					(size 1.27 1.27)
-				)
-				(justify left)
-				(hide yes)
-			)
-		)
-	)
 	(global_label "CPU_D1"
 		(shape bidirectional)
@@
 	(symbol
 		(lib_id "power:GND")
+		(at 201.93 85.09 90)
+		(unit 1)
+		(exclude_from_sim no)
+		(in_bom yes)
+		(on_board yes)
+		(dnp no)
+		(fields_autoplaced yes)
+		(property "Reference" "#PWR039"
+			(at 208.28 85.09 0)
+			(effects
+				(font
+					(size 1.27 1.27)
+				)
+				(hide yes)
+			)
+		)
+		(property "Value" "GND"
+			(at 205.74 85.0899 90)
+			(effects
+				(font
+					(size 1.27 1.27)
+				)
+				(justify right)
+			)
+		)
+		(property "Footprint" ""
+			(at 201.93 85.09 0)
+			(effects
+				(font
+					(size 1.27 1.27)
+				)
+				(hide yes)
+			)
+		)
+		(property "Datasheet" ""
+			(at 201.93 85.09 0)
+			(effects
+				(font
+					(size 1.27 1.27)
+				)
+				(hide yes)
+			)
+		)
+		(property "Description" "Power symbol creates a global label with name \"GND\" , ground"
+			(at 201.93 85.09 0)
+			(effects
+				(font
+					(size 1.27 1.27)
+				)
+				(hide yes)
+			)
+		)
+		(pin "1"
+		)
+		(instances
+			(project "mud-16"
+				(path "/3d8021b6-90cd-4266-8f06-7191a8990bcc/602aecc5-f267-4d0f-9482-a085bf637d86"
+					(reference "#PWR039")
+					(unit 1)
+				)
+			)
+		)
+	)
+	(symbol
+		(lib_id "power:GND")
 		(at 72.39 171.45 90)
 		(unit 1)
@@
 					(unit 1)
 				)
+			)
+		)
+	)
+	(symbol
+		(lib_id "power:GND")
+		(at 179.07 85.09 270)
+		(unit 1)
+		(exclude_from_sim no)
+		(in_bom yes)
+		(on_board yes)
+		(dnp no)
+		(fields_autoplaced yes)
+		(property "Reference" "#PWR062"
+			(at 172.72 85.09 0)
+			(effects
+				(font
+					(size 1.27 1.27)
+				)
+				(hide yes)
+			)
+		)
+		(property "Value" "GND"
+			(at 175.26 85.0899 90)
+			(effects
+				(font
+					(size 1.27 1.27)
+				)
+				(justify right)
+			)
+		)
+		(property "Footprint" ""
+			(at 179.07 85.09 0)
+			(effects
+				(font
+					(size 1.27 1.27)
+				)
+				(hide yes)
+			)
+		)
+		(property "Datasheet" ""
+			(at 179.07 85.09 0)
+			(effects
+				(font
+					(size 1.27 1.27)
+				)
+				(hide yes)
+			)
+		)
+		(property "Description" "Power symbol creates a global label with name \"GND\" , ground"
+			(at 179.07 85.09 0)
+			(effects
+				(font
+					(size 1.27 1.27)
+				)
+				(hide yes)
+			)
+		)
+		(pin "1"
+		)
+		(instances
+			(project "mud-16"
+				(path "/3d8021b6-90cd-4266-8f06-7191a8990bcc/602aecc5-f267-4d0f-9482-a085bf637d86"
+					(reference "#PWR062")
+					(unit 1)
+				)

Commit message: almost done routing
Connections:
- net 1V8_BGACK: now also U14.6 (A4); no longer U14.5 (A3)
- net 1V8_BR: now also U14.7 (A5); no longer U14.4 (A2)
- net 1V8_CLK: now also U14.4 (A2); no longer U14.7 (A5)
- net 1V8_CPU_OE: now also U14.5 (A3); no longer U14.6 (A4)
- net 1V8_DTACK: now also U14.8 (A6); no longer U14.3 (A1)
- net 1V8_LED: now also U14.3 (A1); no longer U14.8 (A6)
- net CLK: now also U14.20 (B2); no longer U14.17 (B5)
- net CPU_BGACK: now also U14.18 (B4); no longer U14.19 (B3)
- net CPU_BR: now also U14.17 (B5); no longer U14.20 (B2)
- net CPU_DTACK: now also U14.16 (B6); no longer U14.21 (B1)
- net CPU_OE: now also U14.19 (B3); no longer U14.18 (B4)
- net at R24.2: now also U14.21 (B1); no longer U14.16 (B6)
Other:
- moved on the sheet: C39, C40, D1, R24
