File: pcb/mud-16.kicad_pcb (KiCad board)
At the start: 4 copper layers, 90 x 100 mm, 100 parts, among them J1 Conn_01x40_MountingPin, J2 Conn_01x06_Pin, J3 Conn_01x02_Pin, U1 74LVC1G04, U10 74HC595, U11 74HC165, U12 74HC165, U13 SN74LVC8T245, U14 SN74LVC8T245, U15 74LVC1G04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

Commit message: routing pcb
Parts:
- J1, R18, U14, U2, U5, U6, U9: moved to F.Cu
- R19, U4, U7: moved to B.Cu
- moved C33 81.6 mm to (162.3, 73.4)
- moved C35 81.6 mm to (158.5, 73.5)
- moved C22 81.6 mm to (158.3, 66.1)
- moved C24 77.4 mm to (162.3, 71.2), turned to 0 degrees
- moved U5 57.1 mm to (117.2, 64.7), turned to 0 degrees
- moved J1 54.8 mm to (51.7, 65.5), turned to 90 degrees
- moved C19 50.5 mm to (21.6, 104.6)
- moved C20 50.5 mm to (25.4, 104.6)
- moved R18 47.5 mm to (58.9, 98.0), turned to 180 degrees
- moved C23 47.0 mm to (145.5, 62.2)
- moved C9 47.0 mm to (149.4, 62.2)
- moved C1 44.3 mm to (137.7, 80.3)
- moved C4 44.3 mm to (142.5, 80.3)
- moved C26 44.3 mm to (146.1, 79.2)
- moved C10 44.0 mm to (29.5, 84.1)
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Connections:
- CPU1 pad 44: CPU_A16 -> unconnected-(CPU1-A16-Pad44)
- U10 pad 3: A12 -> A15
- U10 pad 4: A13 -> A14
- U10 pad 5: A14 -> A13
- U10 pad 6: A15 -> A12
- U10 pad 7: A16 -> unconnected-(U10-QH-Pad7)
- U3 pad 1: D0 -> D7
- U3 pad 2: D1 -> D6
- U3 pad 3: D2 -> D5
- U3 pad 4: D3 -> D4
- U3 pad 5: D4 -> D3
- U3 pad 6: D5 -> D2
- U3 pad 7: D6 -> D1
- U3 pad 8: D7 -> D0
- U5 pad 10: CPU_A16 -> GND
- U5 pad 14: A16 -> GND
Routing:
- net CPU_OE: track 0.00 -> 173.2 mm, vias 0 -> 8
- net CPU_R/W: track 0.00 -> 114.0 mm, vias 0 -> 1
- net A14: track 0.00 -> 92.3 mm, vias 0 -> 3
- net A12: track 0.00 -> 83.6 mm, vias 0 -> 4
- net D7: track 0.00 -> 83.3 mm, vias 0 -> 1
- net D3: track 0.00 -> 82.3 mm, vias 0 -> 1
- net D6: track 0.00 -> 82.1 mm, vias 0 -> 1
- net D5: track 0.00 -> 81.1 mm, vias 0 -> 1
- net D4: track 0.00 -> 80.8 mm, vias 0 -> 1
- net D0: track 0.00 -> 79.9 mm, vias 0 -> 1
- net A13: track 0.00 -> 79.6 mm, vias 0 -> 3
- net D1: track 0.00 -> 79.4 mm, vias 0 -> 1
- net D2: track 0.00 -> 78.5 mm, vias 0 -> 3
- net CPU_D4: track 0.00 -> 65.9 mm
- net CPU_D3: track 0.00 -> 64.1 mm
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
Commit message: almost done routing
Parts:
- C1, C29, C30, C4: moved to F.Cu
- C11, C12: moved to B.Cu
- moved C9 105.9 mm to (45.5, 82.8), turned to 90 degrees
- moved C23 101.5 mm to (45.5, 79.0), turned to -90 degrees
- moved C11 86.6 mm to (113.3, 56.1), turned to 90 degrees
- moved C12 86.6 mm to (111.3, 56.1), turned to -90 degrees
- moved C28 64.3 mm to (84.1, 106.9), turned to -90 degrees
- moved C4 63.0 mm to (80.3, 89.7)
- moved C13 50.8 mm to (147.8, 108.2)
- moved U15 43.8 mm to (87.9, 64.8), turned to -90 degrees
- moved C29 40.7 mm to (74.4, 108.0)
- moved C30 40.5 mm to (72.4, 108.0), turned to 90 degrees
- moved C1 37.4 mm to (100.3, 80.5), turned to 0 degrees
- moved R18 17.5 mm to (73.7, 88.6), turned to 90 degrees
- moved C38 0.49 mm to (73.7, 94.2)
- moved C8 0.49 mm to (76.9, 99.6)
- moved U19 0.49 mm to (79.1, 94.7)
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Connections:
- R24 pad 2: Net-(U14-B6) -> Net-(U14-B1)
- U14 pad 16: Net-(U14-B6) -> CPU_DTACK
- U14 pad 17: CLK -> CPU_BR
- U14 pad 18: CPU_OE -> CPU_BGACK
- U14 pad 19: CPU_BGACK -> CPU_OE
- U14 pad 20: CPU_BR -> CLK
- U14 pad 21: CPU_DTACK -> Net-(U14-B1)
- U14 pad 3: 1V8_DTACK -> 1V8_LED
- U14 pad 4: 1V8_BR -> 1V8_CLK
- U14 pad 5: 1V8_BGACK -> 1V8_CPU_OE
- U14 pad 6: 1V8_CPU_OE -> 1V8_BGACK
- U14 pad 7: 1V8_CLK -> 1V8_BR
- U14 pad 8: 1V8_LED -> 1V8_DTACK
Routing:
- net 3V3: track 0.00 -> 266.6 mm, vias 0 -> 13
- net ADDR_SER: track 0.00 -> 126.0 mm, vias 0 -> 5
- net INPUT_CLK: track 0.00 -> 123.0 mm, vias 0 -> 3
- net INPUT_SH_LD: track 0.00 -> 113.6 mm, vias 0 -> 4
- net R/W: track 0.00 -> 110.2 mm, vias 0 -> 2
- net ADDR_CLR: track 0.00 -> 95.6 mm, vias 0 -> 5
- net ADDR_SRCLK: track 0.00 -> 90.5 mm, vias 0 -> 3
- net /Input Sheet/BTNSTART: track 0.00 -> 88.6 mm, vias 0 -> 5
- net INPUT_QH: track 0.00 -> 85.2 mm, vias 0 -> 2
- net UDS: track 0.00 -> 78.8 mm, vias 0 -> 3
- net LDS: track 0.00 -> 74.0 mm, vias 0 -> 5
- net ADDR_OE: track 0.00 -> 72.3 mm, vias 0 -> 3
- net ADDR_RCLK: track 0.00 -> 68.8 mm, vias 0 -> 6
- net /Input Sheet/BTNMENU: track 0.00 -> 67.9 mm, vias 0 -> 1
- net BTNRST: track 0.00 -> 63.6 mm, vias 0 -> 3
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Other:
- board text added: "a retro console with (mostly) retro components"

Commit message: finish routing
Parts:
- C10, C25: moved to B.Cu
- moved C24 102.2 mm to (60.5, 63.2)
- moved C33 96.5 mm to (66.0, 66.5), turned to 90 degrees
- moved C10 81.7 mm to (110.0, 70.4), turned to 0 degrees
- moved C35 71.0 mm to (87.6, 68.8), turned to 180 degrees
- moved C13 58.7 mm to (116.3, 58.7)
- moved R23 53.3 mm to (58.4, 110.0), turned to -90 degrees
- moved C22 50.8 mm to (107.4, 67.6)
- moved C36 49.3 mm to (60.2, 66.5), turned to -90 degrees
- moved R22 49.1 mm to (55.6, 110.0), turned to -90 degrees
- moved C34 44.0 mm to (60.2, 70.3), turned to -90 degrees
- moved C26 38.3 mm to (109.7, 91.4), turned to 180 degrees
- moved C19 38.1 mm to (59.7, 102.6), turned to 90 degrees
- moved C20 34.8 mm to (59.7, 98.8), turned to 90 degrees
- moved C25 5.92 mm to (87.4, 146.1), turned to 0 degrees
- moved C4 0.36 mm to (80.0, 89.9)
Routing:
- net GND: track 0.00 -> 199.5 mm, vias 0 -> 46
- net /Input Sheet/BTNLB: track 0.00 -> 191.6 mm, vias 0 -> 6
- net 5V: track 37.4 -> 171.2 mm, vias 7 -> 26
- net 3V3: track 266.6 -> 395.6 mm, vias 13 -> 28
- net 1V8: track 27.4 -> 42.1 mm, vias 2 -> 4
- net Net-(C24-Pad2): track 0.00 -> 5.49 mm
- net ADDR_RCLK: track 68.8 -> 73.7 mm
- net D14: track 44.5 -> 49.0 mm
- net D15: track 45.4 -> 49.8 mm
- net A14: track 92.1 -> 95.8 mm
- net A9: track 47.2 -> 50.3 mm
- net D13: track 44.6 -> 47.5 mm
- net D12: track 44.5 -> 47.1 mm
- net CPU_OE: track 165.8 -> 168.3 mm, vias 8 -> 9
- net ADDR_CLR: track 95.6 -> 97.9 mm
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